Commit message: robot falling issue exist here hunter2_robot and hunter_robot

File: src/hunter_robot/hunter_description/description/meshes.xacro (robot description, xacro)
@@ -1,35 +1,18 @@
 <?xml version="1.0"?>
-<robot xmlns:xacro="http://www.ros.org/wiki/xacro">
-  <!-- Macro for visual mesh + primitive collision -->
+<robot xmlns:xacro="http://www.ros.org/wiki/xacro" >
   <xacro:macro name="mesh" params="name">
-    <!-- Visual: always use your .dae file -->
     <visual>
       <origin xyz="0 0 0" rpy="0 0 0"/>
       <geometry>
-        <mesh filename="file://$(find hunter_description)/meshes/${name}.dae"/>
+        <mesh filename="file://$(find hunter_description)/meshes/${name}.dae" />
       </geometry>
     </visual>
-    <!-- Collision: replace problematic meshes with simple primitives -->
     <collision>
       <origin xyz="0 0 0" rpy="0 0 0"/>
       <geometry>
-        <!-- Wheels -->
-        <xacro:if value="${name.find('wheel') != -1}">
-          <!-- radius=0.165, width=0.1 -->
-          <cylinder radius="0.165" length="0.10"/>
-        </xacro:if>
-        <!-- Chassis -->
-        <xacro:if value="${name == 'chassis'}">
-          <!-- size = length 0.65 × width 0.58 × height 0.20 -->
-          <box size="0.65 0.58 0.20"/>
-        </xacro:if>
-        <!-- Fallback tiny collision (for links like steering) -->
-        <xacro:if value="${name != 'chassis' and name.find('wheel') == -1}">
-          <box size="0.01 0.01 0.01"/>
-        </xacro:if>
+        <mesh filename="file://$(find hunter_description)/meshes/${name}.dae" />
       </geometry>
     </collision>
   </xacro:macro>
-  <!-- Invisible virtual part used in your steering links -->
   <xacro:macro name="virtual">
     <visual>
@@ -43,11 +26,10 @@
     </visual>
   </xacro:macro>
-  <!-- Friction macro (unchanged) -->
   <xacro:macro name="gazebo_friction" params="reference">
     <gazebo reference="${reference}">
       <mu1 value="1.0"/>
       <mu2 value="0.5"/>
-      <kp value="10000000.0"/>
-      <kd value="1.0"/>
+      <kp value="10000000.0" />
+      <kd value="1.0" />
       <fdir1 value="1 0 0"/>
     </gazebo>
