Commit message: hunter gazebo and simulation fixed( teleop bridge pending)

File: src/hunter2_robot/hunter2_description/urdf/hunter2_base_gazebo.xacro (robot description, xacro)
@@ -2,4 +2,12 @@
 <robot xmlns:xacro="http://www.ros.org/wiki/xacro"
   name="hunter2_base">
+<material name="Black">
+    <color rgba="0 0 0 1" />
+  </material>
+<material name="Aluminum">
+    <color rgba="0.9 0.9 0.95 1"/>   <!-- base color: very light gray/white -->
+    <specular rgba="0.95 0.95 0.95 1"/> <!-- shiny reflection highlight -->
+    <emission rgba="0 0 0 1"/>         <!-- no self-emission -->
+  </material>
 <link name="base_link" />
   <!-- chassis Link -->
@@ -7,5 +15,5 @@
     <inertial>
       <origin
-        xyz="0.0266989327622036 0.000409203500587652 -0.135901124750884"
+        xyz="0 0 0"
         rpy="0 0 0" />
       <mass
@@ -24,11 +32,9 @@
         rpy="0 0 0" />
       <geometry>
-        <!-- <mesh filename="file://$(find hunter2_robot)/hunter2_description/meshes/base_link.STL" /> -->
-        <box size="0.98 0.745 0.38"/> <!-- W x H x D in meters -->
-      </geometry>
-      <material
-        name="">
-        <color
-          rgba="0.792156862745098 0.819607843137255 0.933333333333333 1" />
+        <mesh filename="file://$(find hunter2_robot)/hunter2_description/meshes/base_link.STL" />
+        <!-- <box size="0.98 0.3 0.27"/>  -->
+      </geometry>
+      <material
+        name="Aluminum">
       </material>
     </visual>
@@ -38,5 +44,5 @@
         rpy="0 0 0" />
       <geometry>
-        <box size="0.98 0.745 0.38"/> <!-- W x H x D in meters -->
+        <box size="0.98 0.3 0.27"/>
       </geometry>
     </collision>
@@ -44,5 +50,5 @@
   <!-- chassis joint -->
   <joint name="chassis_joint" type="fixed">
-    <origin xyz="0.8 0 0.5" rpy="0 0 0" />
+    <origin xyz="0 0 0.37" rpy="0 0 0" />
     <parent link="base_link" />
     <child link="chassis" />
@@ -51,8 +57,19 @@
   <link
     name="left_rear_link">
-    <inertial>
-      <origin
-        xyz="-8.826E-05 6.4342E-05 -0.0096491"
-        rpy="0 0 0" />
+    <collision>
+      <geometry>
+        <cylinder radius="0.165" length="0.14"/>
+      </geometry>
+    </collision>
+    <visual>
+      <geometry>
+        <mesh filename="file://$(find hunter2_robot)/hunter2_description/meshes/left_rear_link.STL" />
+        <!-- <cylinder radius="0.165" length="0.14"/> -->
+      </geometry>
+      <material
+        name="Black">
+      </material>
+    </visual>
+    <inertial>
       <mass
         value="7.6692" />
@@ -65,34 +82,12 @@
         izz="0.11067" />
     </inertial>
-    <visual>
-      <origin
-        xyz="0 0 0"
-        rpy="0 0 0" />
-      <geometry>
-        <!-- <mesh filename="file://$(find hunter2_robot)/hunter2_description/meshes/left_rear_link.STL" /> -->
-        <cylinder radius="0.065" length="0.05"/>
-      </geometry>
-      <material
-        name="">
-        <color
-          rgba="0.79216 0.81961 0.93333 1" />
-      </material>
-    </visual>
-    <collision>
-      <origin
-        xyz="0 0 0"
-        rpy="0 0 0" />
-      <geometry>
-        <cylinder radius="0.065" length="0.05"/>
-      </geometry>
-    </collision>
-  </link>
-  <!-- rear left  Link -->
+  </link>
+  <!-- rear left  JOINT -->
   <joint
     name="left_rear_joint"
     type="continuous">
     <origin
-      xyz="-0.28 0.29249 -0.19558"
-      rpy="1.5708 0 0" />
+      xyz="-0.28 0.29249 -0.165"
+      rpy="-1.57 0 0" />
     <parent
       link="chassis" />
@@ -100,14 +95,25 @@
       link="left_rear_link" />
     <axis
-      xyz="0 0 -1" />
-     <dynamics damping="0.0" friction="15"/>
+      xyz="0 0 1 "/>
+     <dynamics damping="0" friction="15"/>
   </joint>
   <!-- right_rear_link -->
   <link
     name="right_rear_link">
-    <inertial>
-      <origin
-        xyz="8.6344E-05 7.4488E-05 0.0097824"
-        rpy="0 0 0" />
+     <collision>
+      <geometry>
+        <cylinder radius="0.165" length="0.14"/>
+      </geometry>
+    </collision>
+     <visual>
+      <geometry>
+        <mesh filename="file://$(find hunter2_robot)/hunter2_description/meshes/right_rear_link.STL" />
+        <!-- <cylinder radius="0.165" length="0.14"/> -->
+      </geometry>
+      <material
+        name="Black">
+      </material>
+    </visual>
+    <inertial>
       <mass
         value="7.7133" />
@@ -120,26 +126,4 @@
         izz="0.11073" />
     </inertial>
-    <visual>
-      <origin
-        xyz="0 0 0"
-        rpy="0 0 0" />
-      <geometry>
-        <!-- <mesh filename="file://$(find hunter2_robot)/hunter2_description/meshes/right_rear_link.STL" /> -->
-        <cylinder radius="0.065" length="0.05"/>
-      </geometry>
-      <material
-        name="">
-        <color
-          rgba="0.79216 0.81961 0.93333 1" />
-      </material>
-    </visual>
-    <collision>
-      <origin
-        xyz="0 0 0"
-        rpy="0 0 0" />
-      <geometry>
-        <cylinder radius="0.065" length="0.05"/>
-      </geometry>
-    </collision>
   </link>
   <!-- right_rear_join-->
@@ -148,6 +132,6 @@
     type="continuous">
     <origin
-      xyz="-0.28018 -0.29251 -0.19558"
-      rpy="1.5708 0.0026575 0" />
+      xyz="-0.28018 -0.29251 -0.165"
+      rpy="-1.57 0 0" />
     <parent
       link="chassis" />
@@ -155,6 +139,6 @@
       link="right_rear_link" />
     <axis
-      xyz="0 0 -1" />
-     <dynamics damping="0.0" friction="15"/>
+      xyz="0 0 1 "/>
+     <dynamics damping="0" friction="15"/>
   </joint>
   <!-- left steer Link -->
@@ -162,7 +146,4 @@
     name="front_steer_left_link">
     <inertial>
-      <origin
-        xyz="-0.012614 1.8116E-05 0.0023132"
-        rpy="0 0 0" />
       <mass
         value="7.8526" />
@@ -175,25 +156,4 @@
         izz="0.11091" />
     </inertial>
-    <visual>
-      <origin
-        xyz="0 0 0"
-        rpy="0 0 0" />
-      <geometry>
-      <cylinder length="0.001" radius="0.005"/>
-      </geometry>
-      <material
-        name="">
-        <color
-          rgba="0.79216 0.81961 0.93333 1" />
-      </material>
-    </visual>
-    <collision>
-      <origin
-        xyz="0 0 0"
-        rpy="0 0 0" />
-      <geometry>
-      <cylinder length="0.001" radius="0.005"/>
-      </geometry>
-    </collision>
   </link>
   <!-- left steer joint -->
@@ -202,6 +162,6 @@
     type="revolute">
     <origin
-      xyz="0.37142 0.29199 -0.1955"
-      rpy="1.5708 0 0" />
+      xyz="0.37142 0.29199 -0.165"
+      rpy="0 0 0" />
     <parent
       link="chassis" />
@@ -209,10 +169,10 @@
       link="front_steer_left_link" />
     <axis
-      xyz="0 1 0" />
+      xyz="0 0 1" />
     <limit
       lower="-0.69"
       upper="0.69"
-      effort="0"
-      velocity="0" />
+      effort="80"
+      velocity="20" />
   </joint>
   <!-- right steer Link -->
@@ -220,7 +180,4 @@
     name="front_steer_right_link">
     <inertial>
-      <origin
-        xyz="-8.9374E-08 1.0997E-07 0.0095958"
-        rpy="0 0 0" />
       <mass
         value="7.696" />
@@ -233,25 +190,4 @@
         izz="0.11068" />
     </inertial>
-    <visual>
-      <origin
-        xyz="0 0 0"
-        rpy="0 0 0" />
-      <geometry>
-      <cylinder length="0.001" radius="0.005"/>
-      </geometry>
-      <material
-        name="">
-        <color
-          rgba="0.79216 0.81961 0.93333 1" />
-      </material>
-    </visual>
-    <collision>
-      <origin
-        xyz="0 0 0"
-        rpy="0 0 0" />
-      <geometry>
-      <cylinder length="0.001" radius="0.005"/>
-      </geometry>
-    </collision>
   </link>
   <!-- right steer Joint -->
@@ -260,6 +196,6 @@
     type="revolute">
     <origin
-      xyz="0.37142 -0.29201 -0.1955"
-      rpy="1.5708 0 0" />
+      xyz="0.37142 -0.29201 -0.165"
+      rpy="0 0 0" />
     <parent
       link="chassis" />
@@ -267,18 +203,29 @@
       link="front_steer_right_link" />
     <axis
-      xyz="0 1 0" />
+      xyz="0 0 1" />
     <limit
       lower="-0.69"
       upper="0.69"
-      effort="0"
-      velocity="0" />
+      effort="80.0"
+      velocity="2.0" />
   </joint>
 <!-- front left wheel Link -->
   <link
     name="front_left_wheel_link">
-    <inertial>
-      <origin
-        xyz="-6.5774E-06 2.0242E-05 -0.0096386"
-        rpy="0 0 0" />
+    <collision>
+      <geometry>
+        <cylinder radius="0.165" length="0.14"/> <!-- radius ~ half wheel diameter, length ~ wheel thickness -->
+      </geometry>
+    </collision>
+    <visual>
+      <geometry>
+        <mesh filename="file://$(find hunter2_robot)/hunter2_description/meshes/front_left_wheel_link.STL" />
+        <!-- <cylinder radius="0.165" length="0.14"/>  -->
+      </geometry>
+      <material
+        name="Black">
+      </material>
+    </visual>
+    <inertial>
       <mass
         value="7.7007" />
@@ -291,26 +238,4 @@
         izz="0.11072" />
     </inertial>
-    <visual>
-      <origin
-        xyz="0 0 0"
-        rpy="0 0 0" />
-      <geometry>
-        <!-- <mesh filename="file://$(find hunter2_robot)/hunter2_description/meshes/front_left_wheel_link.STL" /> -->
-        <cylinder radius="0.065" length="0.05"/> <!-- radius ~ half wheel diameter, length ~ wheel thickness -->
-      </geometry>
-      <material
-        name="">
-        <color
-          rgba="0.79216 0.81961 0.93333 1" />
-      </material>
-    </visual>
-    <collision>
-      <origin
-        xyz="0 0 0"
-        rpy="0 0 0" />
-      <geometry>
-        <cylinder radius="0.065" length="0.05"/> <!-- radius ~ half wheel diameter, length ~ wheel thickness -->
-      </geometry>
-    </collision>
   </link>
   <!-- front left wheel Joint -->
@@ -320,5 +245,5 @@
     <origin
       xyz="0 0 0"
-      rpy="0 0 0" />
+      rpy="-1.57 0 0" />
     <parent
       link="front_steer_left_link" />
@@ -326,14 +251,25 @@
       link="front_left_wheel_link" />
     <axis
-      xyz="0 0 -1" />
-      <dynamics damping="0.0" friction="15"/>
+      xyz="0 0 1 "/>
+      <dynamics damping="0" friction="15"/>
   </joint>
   <!-- front right wheel Link -->
   <link
     name="front_right_wheel_link">
-    <inertial>
-      <origin
-        xyz="-9.1148E-08 1.1284E-07 0.0095049"
-        rpy="0 0 0" />
+    <collision>
+      <geometry>
+        <cylinder radius="0.165" length="0.14"/>
+      </geometry>
+    </collision>
+    <visual>
+      <geometry>
+        <mesh filename="file://$(find hunter2_robot)/hunter2_description/meshes/front_left_wheel_link.STL" />
+        <!-- <cylinder radius="0.165" length="0.14"/> -->
+      </geometry>
+      <material
+        name="Black">
+      </material>
+    </visual>
+    <inertial>
       <mass
         value="7.5613" />
@@ -346,26 +282,4 @@
         izz="0.11054" />
     </inertial>
-    <visual>
-      <origin
-        xyz="0 0 0"
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