Commit message: laser added to gz_ros2control demo and teleop twist stamped added for ackerman driving using keyboard

File: src/gz_ros2_control_demos/urdf/test_ackermann_drive.xacro.urdf (robot description, URDF)
Before this commit: robot ackermann_drive, 8 links, 7 joints
Links:
- added link laser_link; visual mesh filename=file://$(find gz_ros2_control_demos)/urdf/mid-360.stl scale=0.002 0.002 0.002
Joints:
- added joint body_laser_joint: type fixed, parent chassis, child laser_link, origin xyz=0 0 0.35 rpy=0 0 0

File: src/hunter2_robot/hunter2_description/urdf/hunter2_base_gazebo.xacro (robot description, xacro)
@@ -171,6 +171,6 @@
       xyz="0 0 1" />
     <limit
-      lower="-0.69"
-      upper="0.69"
+      lower="-0.436"
+      upper="0.436"
       effort="80"
       velocity="20" />
@@ -205,6 +205,6 @@
       xyz="0 0 1" />
     <limit
-      lower="-0.69"
-      upper="0.69"
+      lower="-0.436"
+      upper="0.436"
       effort="80.0"
       velocity="2.0" />
@@ -298,4 +298,28 @@
       <dynamics damping="0" friction="15"/>
   </joint>
+<gazebo reference="left_rear_link">
+  <mu1>1.2</mu1>        <!-- lateral friction -->
+  <mu2>1.2</mu2>        <!-- longitudinal friction -->
+  <kp>300000</kp>       <!-- contact stiffness -->
+  <kd>3</kd>            <!-- contact damping -->
+</gazebo>
+<gazebo reference="right_rear_link">
+  <mu1>1.2</mu1>
+  <mu2>1.2</mu2>
+  <kp>300000</kp>
+  <kd>3</kd>
+</gazebo>
+<gazebo reference="front_left_wheel_link">
+  <mu1>1.2</mu1>
+  <mu2>1.2</mu2>
+  <kp>300000</kp>
+  <kd>3</kd>
+</gazebo>
+<gazebo reference="front_right_wheel_link">
+  <mu1>1.2</mu1>
+  <mu2>1.2</mu2>
+  <kp>300000</kp>
+  <kd>3</kd>
+</gazebo>
 <xacro:arg name="sim_gazebo" default="classic"/>
 <ros2_control name="GazeboSystem" type="system">
